Commit message: Freeze confined locomotion flat-2 pretraining engineering baseline

File: src/hexapod_mjlab/assets/robots/el_4090/urdf/el_4090_lidar.urdf (robot description, URDF)
Before this commit: robot el_4090_radar, 29 links, 28 joints
Joints:
- joint LIDAR_SENSOR_FIX: origin xyz=0 0.0453 0 rpy=0 0 0 -> xyz=0 0.0453 0 rpy=-1.5707963267948966 0 0
